Commit message: Changed all parameters to Scoutt 2.0's. Design currently only implements 1 Lidar for sensing

File: sensor_kit/scout_sensor_kit_launch/scout_sensor_kit_description/urdf/sensor_kit.xacro (robot description, xacro)
@@ -30,5 +30,5 @@
       />
     </xacro:VLS-128>
-    <xacro:VLP-16 parent="sensor_kit_base_link" name="velodyne_left" topic="/points_raw" hz="10" samples="220" gpu="$(arg gpu)">
+    <!-- <xacro:VLP-16 parent="sensor_kit_base_link" name="velodyne_left" topic="/points_raw" hz="10" samples="220" gpu="$(arg gpu)">
       <origin
         xyz="${calibration['sensor_kit_base_link']['velodyne_left_base_link']['x']}
@@ -49,5 +49,5 @@
              ${calibration['sensor_kit_base_link']['velodyne_right_base_link']['yaw']}"
       />
-    </xacro:VLP-16>
+    </xacro:VLP-16> -->
     <!-- camera -->
     <!-- <xacro:monocular_camera_macro

File: sensor_kit/scout_sensor_kit_launch/scout_sensor_kit_description/urdf/sensors.xacro (robot description, xacro)
@@ -16,5 +16,5 @@
   <!-- embedded sensors -->
   <xacro:include filename="$(find velodyne_description)/urdf/VLP-16.urdf.xacro"/>
-  <xacro:VLP-16 parent="base_link" name="velodyne_rear" topic="velodyne_rear/velodyne_points" hz="10" samples="220" gpu="false">
+  <!-- <xacro:VLP-16 parent="base_link" name="velodyne_rear" topic="velodyne_rear/velodyne_points" hz="10" samples="220" gpu="false">
     <origin
       xyz="${calibration['base_link']['velodyne_rear_base_link']['x']}
@@ -25,4 +25,4 @@
            ${calibration['base_link']['velodyne_rear_base_link']['yaw']}"
     />
-  </xacro:VLP-16>
+  </xacro:VLP-16> -->
 </robot>

File: vehicle/scout_vehicle_launch/scout_vehicle_description/urdf/scout_vehicle.urdf (robot description, URDF)
Before this commit: robot None, 7 links, 6 joints
Links:
- link base_link: geometry collision box size=0.15416666666666667 0.627 0.06999999999999999; collision box size=0.925 0.38 0.21
- link front_left_wheel_link: geometry collision cylinder length=0.11653 radius=0.16459; visual mesh filename=package://robot_description/meshes/scout_v2/wheel_type2.dae
- link front_right_wheel_link: geometry collision cylinder length=0.11653 radius=0.16459; visual mesh filename=package://robot_description/meshes/scout_v2/wheel_type1.dae
- link rear_left_wheel_link: geometry collision cylinder length=0.11653 radius=0.16459; visual mesh filename=package://robot_description/meshes/scout_v2/wheel_type1.dae
- link rear_right_wheel_link: geometry collision cylinder length=0.11653 radius=0.16459; visual mesh filename=package://robot_description/meshes/scout_v2/wheel_type2.dae
Joints:
- joint base_footprint_joint: origin xyz=0 0 -0.23479 rpy=0 0 0 -> xyz=0 0 0.23479 rpy=0 0 0
